File: KiCad/Router-Rebooter.kicad_pcb (KiCad board)
At the start: 2 copper layers, 62 x 49 mm, 14 parts, among them J1 12V Power In, J2 12V Power Out, K1 SRD-05VDC-SL-C, Q1 2N2222, U1 ESP32-C3-Zero, U2 PSU2-5, U3 PSU2-5

Commit message: Added indicator LEDs (OK & FAILURE)
OK is steady green when everything is okay
FAILURE is flashing red when rebooting
Parts:
- added D2: OK, LED_THT:LED_D3.0mm, F.Cu at (108.2, 37.0)
- added D3: FAILURE, LED_THT:LED_D3.0mm, F.Cu at (105.2, 37.0)
- added R2: R, Resistor_THT:R_Axial_DIN0207_L6.3mm_D2.5mm_P7.62mm_Horizontal, F.Cu at (113.2, 64.9)
- added R3: R, Resistor_THT:R_Axial_DIN0207_L6.3mm_D2.5mm_P7.62mm_Horizontal, F.Cu at (109.2, 64.9)
Connections:
- U1 pad 4: unconnected-(U1-IO0-Pad4) -> Net-(U1-IO0)
- U1 pad 5: unconnected-(U1-IO1-Pad5) -> Net-(U1-IO1)
Routing:
- net GND: track 143.3 -> 174.3 mm
- net Net-(D3-A): track 0.00 -> 22.9 mm
- net Net-(D2-A): track 0.00 -> 22.2 mm
- net Net-(U1-IO0): track 0.00 -> 20.7 mm, vias 0 -> 1
- net Net-(U1-IO1): track 0.00 -> 19.3 mm, vias 0 -> 1

Commit message: Cosmetic changes
Routing:
- net +5V_{RELAY}: track 22.0 -> 23.3 mm
Changed lines of the file:
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@@
-	)
-	(segment
-		(start 73.9964 37.6274)
-		(end 79.649085 37.6274)
-		(width 1)
-		(layer "F.Cu")
-		(net 1)
 	)
 	(segment
@@
 	)
 	(segment
-		(start 79.649085 37.6274)
-		(end 83.546399 41.524714)
-		(width 1)
-		(layer "F.Cu")
-		(net 1)
-	)
-	(segment
 		(start 82.2964 51.0074)
 		(end 82.8864 51.5974)
@@
 	)
 	(segment
-		(start 83.546399 41.524714)
+		(start 73.9964 37.6274)
+		(end 81.7964 37.6274)
+		(width 1)
+		(layer "F.Cu")
+		(net 1)
+	)
+	(segment
+		(start 83.546399 39.377399)
 		(end 83.546399 46.237401)
+		(width 1)
+		(layer "F.Cu")
+		(net 1)
+	)
+	(segment
+		(start 81.7964 37.6274)
+		(end 83.546399 39.377399)
 		(width 1)
 		(layer "F.Cu")
@@
 		(min_thickness 0.25)
 		(filled_areas_thickness no)
-		(fill yes
+		(fill
 			(thermal_gap 0.5)
 			(thermal_bridge_width 0.5)

Commit message: Corrected schematic/footprint errors
Parts:
- removed U3: PSU2-5, Package_TO_SOT_THT:TO-220-3_Vertical
- added J2: ESP32 Power Bypass, Connector_PinHeader_2.54mm:PinHeader_1x02_P2.54mm_Vertical, F.Cu at (61.3, 59.5)
- K1: value SRD-05VDC-SL-C -> OMRON G5LE-1-VD; footprint Relay_THT:Relay_SPDT_SANYOU_SRD_Series_Form_C -> Relay_THT:Relay_SPDT_Omron-G5LE-1
- Q1: value 2N2222 -> PN2222A; footprint Package_TO_SOT_THT:TO-92L_Inline -> Package_TO_SOT_THT:TO-92_Inline
- moved Q1 2.48 mm to (98.3, 55.3), turned to 90 degrees
- moved K1 0.07 mm to (80.4, 41.4), turned to 90 degrees
- renumbered J2 to J1, J1 to J3, R2 to R1, R3 to R2, R1 to R3, U2 to U1, U1 to U2
Connections:
- D1 pad 1: +5V_{RELAY} -> /+12V_{IN}
- K1 pad 2: +5V_{RELAY} -> /+12V_{IN}
- K1 pad 3: unconnected-(K1-NO-Pad3) -> (no net)
- Q1 pad 1: Net-(D1-A) -> GND
- Q1 pad 3: GND -> Net-(D1-A)
- U1 pad 3: +5V_{ESP32} -> Net-(J2-Pin_1)
Routing:
- net +5V_{RELAY}: track 23.3 -> 0.00 mm
- net GND: track 174.3 -> 166.3 mm, vias 0 -> 1
- net Net-(J2-Pin_1): track 0.00 -> 6.35 mm
- net +5V_{ESP32}: track 52.4 -> 55.1 mm
- net Net-(U2-IO0): track 20.7 -> 22.9 mm
- net /+12V_{IN}: track 36.1 -> 36.9 mm
Other:
- board text added: "12VDC Relay Coil Normally Closed"
- board text added: "Brett Hallen, Mar 2026"
- board text added: "Brett's Broadband Router Rebooter (Rev. B)"
- board text added: "ESP32 Power Bypass"
- board text removed: "Brett Hallen, Jan 2026"
- board text removed: "Brett's Broadband Router Rebooter (Rev. A)"
