File: KiCad/Router-Rebooter.kicad_pcb (KiCad board)
At the start: 2 copper layers, 62 x 49 mm, 18 parts, among them J1 12V Power Out, J2 ESP32 Power Bypass, J3 12V Power In, K1 OMRON G5LE-1-VD, Q1 PN2222A, U1 PSU2-5, U2 ESP32-C3-Zero

Commit message: Modified component IDs to match
Now R1 is for LED D1, R2 is for LED D2
Parts:
- renumbered D2 to D1, D3 to D2, D1 to D3
Changed lines of the file:
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@@
 			(layers "*.Cu" "*.Mask")
 			(remove_unused_layers no)
-			(net 1 "Net-(D1-A)")
+			(net 8 "Net-(D3-A)")
 			(pinfunction "C")
 			(pintype "passive")
@@
 			(layers "*.Cu" "*.Mask")
 			(remove_unused_layers no)
-			(net 6 "Net-(D2-A)")
+			(net 1 "Net-(D1-A)")
 			(pintype "passive")
 		)
@@
 		(descr "LED, diameter 3.0mm, 2 pins, generated by kicad-footprint-generator")
 		(tags "LED")
-		(property "Reference" "D3"
+		(property "Reference" "D2"
 			(at 1 3 0)
 			(layer "F.SilkS")
@@
 			(layers "*.Cu" "*.Mask")
 			(remove_unused_layers no)
-			(net 8 "Net-(D3-A)")
+			(net 6 "Net-(D2-A)")
 			(pinfunction "A")
 			(pintype "passive")
@@
 		(descr "LED, diameter 3.0mm, 2 pins, generated by kicad-footprint-generator")
 		(tags "LED")
-		(property "Reference" "D2"
+		(property "Reference" "D1"
 			(at 1 -3 0)
 			(layer "F.SilkS")
@@
 			(layers "*.Cu" "*.Mask")
 			(remove_unused_layers no)
-			(net 6 "Net-(D2-A)")
+			(net 1 "Net-(D1-A)")
 			(pinfunction "A")
 			(pintype "passive")
@@
 			(layers "*.Cu" "*.Mask")
 			(remove_unused_layers no)
-			(net 8 "Net-(D3-A)")
+			(net 6 "Net-(D2-A)")
 			(pintype "passive")
 		)
@@
 			(layers "*.Cu" "*.Mask")
 			(remove_unused_layers no)
-			(net 1 "Net-(D1-A)")
+			(net 8 "Net-(D3-A)")
 			(pintype "passive")
 		)
@@
 		(descr "Diode, DO-35_SOD27 series, Axial, Horizontal, pin pitch=7.62mm, length*diameter=4*2mm^2, http://www.diodes.com/_files/packages/DO-35.pdf")
 		(tags "Diode DO-35_SOD27 series Axial Horizontal pin pitch 7.62mm  length 4mm diameter 2mm")
-		(property "Reference" "D1"
+		(property "Reference" "D3"
 			(at -2.69 -1 0)
 			(layer "F.SilkS")
@@
 			(layers "*.Cu" "*.Mask")
 			(remove_unused_layers no)
-			(net 1 "Net-(D1-A)")
+			(net 8 "Net-(D3-A)")
 			(pinfunction "A")
 			(pintype "passive")
@@
 	)
 	(segment
-		(start 91.7764 52.8674)
-		(end 90.5064 51.5974)
-		(width 1)
-		(layer "F.Cu")
-		(net 1)
-	)
-	(segment
-		(start 90.5064 43.6974)
-		(end 90.5064 51.5974)
-		(width 1)
-		(layer "F.Cu")
-		(net 1)
-	)
-	(segment
-		(start 91.8374 52.8064)
-		(end 98.2534 52.8064)
-		(width 1)
+		(start 109.6174 38.1864)
+		(end 109.6174 53.6384)
+		(width 0.2)
 		(layer "F.Cu")
 		(net 1)
 	)
 	(segment
-		(start 91.7764 52.8674)
-		(end 91.8374 52.8064)
-		(width 1)
+		(start 109.6174 53.6384)
+		(end 113.2164 57.2374)
+		(width 0.2)
 		(layer "F.Cu")
 		(net 1)
 	)
 	(segment
-		(start 82.2964 35.4874)
-		(end 90.5064 43.6974)
-		(width 1)
+		(start 110.7564 37.0474)
+		(end 109.6174 38.1864)
+		(width 0.2)
 		(layer "F.Cu")
 		(net 1)
@@
 	)
 	(segment
-		(start 109.6174 38.1864)
-		(end 109.6174 53.6384)
-		(width 0.2)
-		(layer "F.Cu")
-		(net 6)
-	)
-	(segment
-		(start 109.6174 53.6384)
-		(end 113.2164 57.2374)
+		(start 109.2164 43.5874)
+		(end 109.2164 57.2374)
 		(width 0.2)
 		(layer "F.Cu")
@@
 	)
 	(segment
-		(start 110.7564 37.0474)
-		(end 109.6174 38.1864)
+		(start 102.6764 37.0474)
+		(end 109.2164 43.5874)
 		(width 0.2)
 		(layer "F.Cu")
@@
 	)
 	(segment
-		(start 109.2164 43.5874)
-		(end 109.2164 57.2374)
-		(width 0.2)
+		(start 91.7764 52.8674)
+		(end 90.5064 51.5974)
+		(width 1)
 		(layer "F.Cu")
 		(net 8)
 	)
 	(segment
-		(start 102.6764 37.0474)
-		(end 109.2164 43.5874)
-		(width 0.2)
+		(start 90.5064 43.6974)
+		(end 90.5064 51.5974)
+		(width 1)
+		(layer "F.Cu")
+		(net 8)
+	)
+	(segment
+		(start 91.8374 52.8064)
+		(end 98.2534 52.8064)
+		(width 1)
+		(layer "F.Cu")
+		(net 8)
+	)
+	(segment
+		(start 91.7764 52.8674)
+		(end 91.8374 52.8064)
+		(width 1)
+		(layer "F.Cu")
+		(net 8)
+	)
+	(segment
+		(start 82.2964 35.4874)
+		(end 90.5064 43.6974)
+		(width 1)
 		(layer "F.Cu")
 		(net 8)
