File: KiCad/Router-Rebooter.kicad_sch (KiCad schematic)
At the start: 14 parts, among them J1 12V Power In, J2 12V Power Out, K1 SRD-05VDC-SL-C, Q1 2N2222, U1 ESP32-C3-Zero, U2 PSU2-5, U3 PSU2-5

Commit message: Added indicator LEDs (OK & FAILURE)
OK is steady green when everything is okay
FAILURE is flashing red when rebooting
Parts:
- added D2: OK, LED_THT:LED_D3.0mm, symbol Device:LED
- added D3: FAILURE, LED_THT:LED_D3.0mm, symbol Device:LED
- added R2, R3: R, Resistor_THT:R_Axial_DIN0207_L6.3mm_D2.5mm_P7.62mm_Horizontal, symbol Device:R
Connections:
- net GND: now also D2.1 (K), D3.1 (K)
- net at U1.4 (IO0): now also R2.1
- net at U1.5 (IO1): now also R3.1
- new net: D3.2 (A), R3.2
- new net: D2.2 (A), R2.2
- no-connect marks 16 -> 14
Other:
- moved on the sheet: R1

Commit message: Cosmetic changes
Other:
- moved on the sheet: H1, H2, H3, H4, J1, U2, U3

Commit message: Corrected schematic/footprint errors
Parts:
- removed K1: SRD-05VDC-SL-C, Relay_THT:Relay_SPDT_SANYOU_SRD_Series_Form_C, symbol Relay:SANYOU_SRD_Form_C
- removed Q1: 2N2222, Package_TO_SOT_THT:TO-92L_Inline, symbol Simulation_SPICE:NPN
- removed U3: PSU2-5, Package_TO_SOT_THT:TO-220-3_Vertical, symbol Regulator_Linear:LM7805_TO220
- added J2: ESP32 Power Bypass, Connector_PinHeader_2.54mm:PinHeader_1x02_P2.54mm_Vertical, symbol Connector_Generic:Conn_01x02
- added K1: OMRON G5LE-1-VD, Relay_THT:Relay_SPDT_Omron-G5LE-1, symbol Relay:SANYOU_SRD_Form_B
- added Q1: PN2222A, Package_TO_SOT_THT:TO-92_Inline, symbol Transistor_BJT:PN2222A
- renumbered J2 to J1, J1 to J3, R2 to R1, R3 to R2, R1 to R3, U2 to U1, U1 to U2
Connections:
- net +5V_{RELAY} is gone; now on net +12V_{IN}: D1.1 (K)
- net +12V_{IN}: now also K1.1, K1.2
- net +12V_{OUT}: now also K1.4
- net +5V_{ESP32}: now also J2.2 (Pin_2); no longer U1.3 (VO)
- net GND: now also Q1.1 (E)
- net at D1.2 (A): now also K1.5, Q1.3 (C)
- net at R3.2: now also Q1.2 (B)
- new net: J2.1 (Pin_1), U1.3 (VO)
- no-connect marks 14 -> 13
