File: KiCad/Router-Rebooter.kicad_sch (KiCad schematic)
At the start: 18 parts, among them J1 12V Power Out, J2 ESP32 Power Bypass, J3 12V Power In, K1 OMRON G5LE-1-VD, Q1 PN2222A, U1 PSU2-5, U2 ESP32-C3-Zero

Commit message: Modified component IDs to match
Now R1 is for LED D1, R2 is for LED D2
Parts:
- renumbered D2 to D1, D3 to D2, D1 to D3
Changed lines of the file:
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@@
 		(on_board yes)
 		(dnp no)
-		(property "Reference" "D3"
+		(property "Reference" "D2"
 			(at 99.822 89.916 0)
 			(effects
@@
 			(project ""
 				(path "/8de648ee-e13b-40be-adc8-7d40ce8ea697"
-					(reference "D3")
+					(reference "D2")
 					(unit 1)
 				)
@@
 		(dnp no)
 		(fields_autoplaced yes)
-		(property "Reference" "D1"
+		(property "Reference" "D3"
 			(at 148.59 58.42 0)
 			(effects
@@
 			(project "Router-Rebooter"
 				(path "/8de648ee-e13b-40be-adc8-7d40ce8ea697"
-					(reference "D1")
+					(reference "D3")
 					(unit 1)
 				)
@@
 		(on_board yes)
 		(dnp no)
-		(property "Reference" "D2"
+		(property "Reference" "D1"
 			(at 85.09 88.392 0)
 			(effects
@@
 			(project ""
 				(path "/8de648ee-e13b-40be-adc8-7d40ce8ea697"
-					(reference "D2")
-					(unit 1)
-				)
+					(reference "D1")
+					(unit 1)
+				)
