File: KiCad/RevD/Router-Rebooter.kicad_pcb (KiCad board)
At the start: 2 copper layers, 62 x 49 mm, 18 parts, among them J1 12V Out, J3 12V In, K1 OMRON G5LE-1-VD, Q1 PN2222A, U1 PSU2-5, U2 ESP32-C3-Zero

Commit message: Modified ESP32 power bypass
The ESP32 serial via USB wouldn't connect if the board was already powered via 12V - had to connect via USB first and then apply 12V power.
So let's just have a simple 2-pin header to connect or disconnect the 5V regulator from the ESP32.
Parts:
- removed D4: 1N5819, Diode_THT:D_DO-41_SOD81_P10.16mm_Horizontal
- added J2: ESP32 Power, Connector_PinHeader_2.54mm:PinHeader_1x02_P2.54mm_Vertical, F.Cu at (116.0, 61.2)
Routing:
- net +5V_{ESP32}: track 56.4 -> 64.0 mm
Other:
- board text added: "Brett Hallen, May 2026"
- board text added: "Brett's Router Rebooter (Rev. D)"
- board text removed: "Brett Hallen, Apr 2026"
- board text removed: "Brett's Router Rebooter (Rev. C)"
