File: KiCad/RevD/Router-Rebooter.kicad_sch (KiCad schematic)
At the start: 18 parts, among them J1 12V Out, J3 12V In, K1 OMRON G5LE-1-VD, Q1 PN2222A, U1 PSU2-5, U2 ESP32-C3-Zero

Commit message: Modified ESP32 power bypass
The ESP32 serial via USB wouldn't connect if the board was already powered via 12V - had to connect via USB first and then apply 12V power.
So let's just have a simple 2-pin header to connect or disconnect the 5V regulator from the ESP32.
Parts:
- removed D4: 1N5819, Diode_THT:D_DO-41_SOD81_P10.16mm_Horizontal, symbol Device:D
- added J2: ESP32 Power, Connector_PinHeader_2.54mm:PinHeader_1x02_P2.54mm_Vertical, symbol Connector_Generic:Conn_01x02
Connections:
- net +5V_{ESP32}: now also J2.2 (Pin_2)
- net at U1.3 (VO): now also J2.1 (Pin_1)
Changed lines of the file:
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@@
 	(title_block
 		(title "Broadband Router Rebooter")
-		(date "28/MAR/2026")
-		(rev "C")
+		(date "1/MAY/2026")
+		(rev "D")
 		(company "Brett Hallen")
 	)
@@
 		)
 	)
-	(text_box "Schottky diode prevents regulator back-feeding when USB is connected."
+	(text_box "Prevent regulator from powering ESP32 when USB connected."
 		(exclude_from_sim no)
 		(at 193.04 63.5 0)
-		(size 73.66 3.81)
+		(size 62.23 3.81)
 		(margins 0.9525 0.9525 0.9525 0.9525)
 		(stroke
@@
 	(wire
 		(pts
+			(xy 223.52 77.47) (xy 240.03 77.47)
+		)
+		(stroke
+			(width 0)
+			(type default)
+		)
+	)
+	(wire
+		(pts
 			(xy 190.5 77.47) (xy 199.39 77.47)
 		)
@@
 	(wire
 		(pts
-			(xy 226.06 77.47) (xy 240.03 77.47)
-		)
-		(stroke
-			(width 0)
-			(type default)
-		)
-	)
-	(wire
-		(pts
 			(xy 68.58 111.76) (xy 71.12 111.76)
 		)
@@
 	(wire
 		(pts
-			(xy 218.44 77.47) (xy 214.63 77.47)
+			(xy 214.63 77.47) (xy 220.98 77.47)
 		)
 		(stroke
@@
 			)
 			(justify left bottom)
+		)
+	)
+	(symbol
+		(lib_id "Connector_Generic:Conn_01x02")
+		(at 220.98 72.39 90)
+		(unit 1)
+		(exclude_from_sim no)
+		(in_bom yes)
+		(on_board yes)
+		(dnp no)
+		(fields_autoplaced yes)
+		(property "Reference" "J2"
+			(at 226.06 71.1199 90)
+			(effects
+				(font
+					(size 1.27 1.27)
+				)
+				(justify right)
+			)
+		)
+		(property "Value" "ESP32 Power"
+			(at 226.06 73.6599 90)
+			(effects
+				(font
+					(size 1.27 1.27)
+				)
+				(justify right)
+			)
+		)
+		(property "Footprint" "Connector_PinHeader_2.54mm:PinHeader_1x02_P2.54mm_Vertical"
+			(at 220.98 72.39 0)
+			(effects
+				(font
+					(size 1.27 1.27)
+				)
+				(hide yes)
+			)
+		)
+		(property "Datasheet" "~"
+			(at 220.98 72.39 0)
+			(effects
+				(font
+					(size 1.27 1.27)
+				)
+				(hide yes)
+			)
+		)
+		(property "Description" "Generic connector, single row, 01x02, script generated (kicad-library-utils/schlib/autogen/connector/)"
+			(at 220.98 72.39 0)
+			(effects
+				(font
+					(size 1.27 1.27)
+				)
+				(hide yes)
+			)
+		)
+		(pin "2"
+		)
+		(pin "1"
+		)
+		(instances
+			(project ""
+				(path "/8de648ee-e13b-40be-adc8-7d40ce8ea697"
+					(reference "J2")
+					(unit 1)
+				)
+			)
 		)
 	)
@@
 					(unit 1)
 				)
-			)
-		)
-	)
-	(symbol
-		(lib_id "Device:D")
-		(at 222.25 77.47 180)
-		(unit 1)
-		(exclude_from_sim no)
-		(in_bom yes)
-		(on_board yes)
-		(dnp no)
-		(fields_autoplaced yes)
-		(property "Reference" "D4"
-			(at 222.25 71.12 0)
-			(effects
-				(font
-					(size 1.27 1.27)
-				)
-			)
-		)
-		(property "Value" "1N5819"
-			(at 222.25 73.66 0)
-			(effects
-				(font
-					(size 1.27 1.27)
-				)
-			)
-		)
-		(property "Footprint" "Diode_THT:D_DO-41_SOD81_P10.16mm_Horizontal"
-			(at 222.25 77.47 0)
-			(effects
-				(font
-					(size 1.27 1.27)
-				)
-				(hide yes)
-			)
-		)
-		(property "Datasheet" "~"
-			(at 222.25 77.47 0)
-			(effects
-				(font
-					(size 1.27 1.27)
-				)
-				(hide yes)
-			)
-		)
-		(property "Description" "Diode"
-			(at 222.25 77.47 0)
-			(effects
-				(font
-					(size 1.27 1.27)
-				)
-				(hide yes)
-			)
-		)
-		(property "Sim.Device" "D"
-			(at 222.25 77.47 0)
-			(effects
-				(font
-					(size 1.27 1.27)
-				)
-				(hide yes)
-			)
-		)
-		(property "Sim.Pins" "1=K 2=A"
-			(at 222.25 77.47 0)
-			(effects
-				(font
-					(size 1.27 1.27)
-				)
-				(hide yes)
-			)
-		)
-		(pin "1"
-		)
-		(pin "2"
-		)
-		(instances
-			(project "Router-Rebooter"
-				(path "/8de648ee-e13b-40be-adc8-7d40ce8ea697"
-					(reference "D4")
-					(unit 1)
-				)
